Commit message: fix: virtual joints for solver

File: open_manipulator_x_moveit_config/config/open_manipulator_x.ros2_control.xacro (robot description, xacro)
@@ -42,4 +42,18 @@
         <state_interface name="velocity"/>
       </joint>
+      <joint name="virtual_roll_joint">
+        <command_interface name="position"/>
+        <state_interface name="position">
+          <param name="initial_value">${initial_positions['virtual_roll_joint']}</param>
+        </state_interface>
+        <state_interface name="velocity"/>
+      </joint>
+      <joint name="virtual_yaw_joint">
+        <command_interface name="position"/>
+        <state_interface name="position">
+          <param name="initial_value">${initial_positions['virtual_yaw_joint']}</param>
+        </state_interface>
+        <state_interface name="velocity"/>
+      </joint>
     </ros2_control>
   </xacro:macro>
